File: hardware/pcb/hitteStress21-pcb/hitteStress21-pcb.kicad_pcb (KiCad board)
At the start: 2 copper layers, 70 x 115 mm, 21 parts, among them J1 Conn_01x02_Female, J2 Conn_01x05, J3 Conn_01x03, J4 Conn_01x02, U1 HTCC-AB01, U2 GPS

Commit message: Update PCB
Parts:
- moved J1 52.7 mm to (186.4, 52.8), turned to 180 degrees
- moved R3 48.7 mm to (194.1, 102.6)
- moved R2 48.7 mm to (194.1, 99.6)
- moved R1 48.6 mm to (194.1, 96.5)
- moved C1 43.5 mm to (174.8, 110.2), turned to 90 degrees
- moved TH1 38.7 mm to (186.4, 69.1), turned to 90 degrees
- moved PSU2 36.1 mm to (229.9, 50.3)
- moved U2 33.0 mm to (223.5, 81.8)
- moved U1 28.7 mm to (212.3, 101.1)
- moved J3 28.7 mm to (169.2, 107.7)
- moved R4 28.2 mm to (194.1, 105.7)
- moved J2 28.0 mm to (171.7, 87.4)
- moved J4 18.5 mm to (169.2, 70.6)
- moved PSU1 7.26 mm to (191.0, 81.8), turned to 90 degrees
- moved G*** 1.91 mm to (195.6, 126.4)
Routing:
- net GND: track 0.00 -> 195.5 mm, vias 0 -> 90
- net /PV: track 0.00 -> 87.2 mm
- net /3V3: track 0.00 -> 78.4 mm
- net /AM2305_DATA: track 0.00 -> 62.3 mm
- net /5V: track 0.00 -> 45.6 mm, vias 0 -> 1
- net /3V3_EXT: track 0.00 -> 39.4 mm
- net /GPS_RXD: track 0.00 -> 39.0 mm
- net /GPS_TXD: track 0.00 -> 36.8 mm
- net /PM_RX: track 0.00 -> 27.3 mm
- net /PM_TX: track 0.00 -> 27.1 mm
- net Net-(J2-Pad4): track 0.00 -> 25.6 mm
- net /5V_EXT: track 0.00 -> 24.5 mm, vias 0 -> 1
- net /SDS011_RXD: track 0.00 -> 24.2 mm
- net /SDS011_TXD: track 0.00 -> 20.8 mm
- net Net-(J1-Pad1): track 38.7 -> 26.9 mm
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- added copper zone on B.Cu, net GND
- added copper zone on F.Cu, net GND
Other:
- board size 70 x 115 mm -> 69 x 115 mm
- board text added: "20210407"
- board text added: "Stichting IoT Apeldoorn e/o www.iotapeldoorn.nl"
- board text removed: "20210406"
- board text removed: "Stichting IoT Apeldoorn e/o www.iot-apeldoorn.ml"
