File: hardware/pcb/hitteStress21-pcb/hitteStress21-pcb.sch (KiCad schematic (older format))
At the start: 13 parts, among them J1 Conn_01x02_Female, J2 Conn_01x05, J3 Conn_01x03, U1 HTCC-AB01, U2 GPS

Commit message: PCB design step
Parts:
- C1: footprint (none) -> Resistor_THT:R_Axial_DIN0204_L3.6mm_D1.6mm_P5.08mm_Horizontal
- J1: footprint (none) -> Connector_Phoenix_MC_HighVoltage:PhoenixContact_MCV_1,5_2-G-5.08_1x02_P5.08mm_Vertical
- J2: footprint (none) -> hitteStress21-pcb:JST_XH_S5B-XH-A_1x05_P2.50mm_Horizontal
- J3, PSU1: footprint (none) -> Connector_PinHeader_2.54mm:PinHeader_1x03_P2.54mm_Vertical
- PSU2: footprint (none) -> hitteStress21-pcb:IRM-03
- R1, R2, R3, R4: footprint (none) -> Resistor_THT:R_Axial_DIN0204_L3.6mm_D1.6mm_P7.62mm_Horizontal
- TH1: footprint (none) -> Resistor_THT:R_Axial_DIN0207_L6.3mm_D2.5mm_P7.62mm_Horizontal
- U1: footprint (none) -> hitteStress21-pcb:HTCC-AB01
- U2: footprint (none) -> hitteStress21-pcb:GPS
Changed lines of the file:
@@
 F 0 "PSU2" H 3100 2365 50  0000 C CNN
 F 1 "IRM-03" H 3100 2274 50  0000 C CNN
-F 2 "" H 3100 2050 50  0001 C CNN
+F 2 "hitteStress21-pcb:IRM-03" H 3100 2050 50  0001 C CNN
 F 3 "" H 3100 2050 50  0001 C CNN
 	1    3100 2000
@@
 F 0 "PSU1" H 1950 5665 50  0000 C CNN
 F 1 "MINIDCDCBOOST5V" H 1950 5574 50  0000 C CNN
-F 2 "" H 1950 5250 50  0001 C CNN
+F 2 "Connector_PinHeader_2.54mm:PinHeader_1x03_P2.54mm_Vertical" H 1950 5250 50  0001 C CNN
 F 3 "" H 1950 5250 50  0001 C CNN
 	1    1950 5250
@@
 F 0 "J1" H 1392 1725 50  0000 C CNN
 F 1 "Conn_01x02_Female" H 1392 1816 50  0000 C CNN
-F 2 "" H 1500 2050 50  0001 C CNN
+F 2 "Connector_Phoenix_MC_HighVoltage:PhoenixContact_MCV_1,5_2-G-5.08_1x02_P5.08mm_Vertical" H 1500 2050 50  0001 C CNN
 F 3 "~" H 1500 2050 50  0001 C CNN
 	1    1500 2050
@@
 F 0 "TH1" V 2058 1900 50  0000 C CNN
 F 1 "Thermistor" V 2149 1900 50  0000 C CNN
-F 2 "" H 2300 1900 50  0001 C CNN
+F 2 "Resistor_THT:R_Axial_DIN0207_L6.3mm_D2.5mm_P7.62mm_Horizontal" H 2300 1900 50  0001 C CNN
 F 3 "~" H 2300 1900 50  0001 C CNN
 	1    2300 1900
@@
 F 0 "U1" H 6450 3265 50  0000 C CNN
 F 1 "HTCC-AB01" H 6450 3174 50  0000 C CNN
-F 2 "" H 6450 2450 50  0001 C CNN
+F 2 "hitteStress21-pcb:HTCC-AB01" H 6450 2450 50  0001 C CNN
 F 3 "" H 6450 2450 50  0001 C CNN
 	1    6450 2400
@@
 F 0 "J2" H 4830 5292 50  0000 L CNN
 F 1 "Conn_01x05" H 4830 5201 50  0000 L CNN
-F 2 "" H 4750 5250 50  0001 C CNN
+F 2 "hitteStress21-pcb:JST_XH_S5B-XH-A_1x05_P2.50mm_Horizontal" H 4750 5250 50  0001 C CNN
 F 3 "~" H 4750 5250 50  0001 C CNN
 	1    4750 5250
@@
 F 0 "R1" V 4000 4950 50  0000 C CNN
 F 1 "1k" V 4000 5100 50  0000 C CNN
-F 2 "" V 4030 5050 50  0001 C CNN
+F 2 "Resistor_THT:R_Axial_DIN0204_L3.6mm_D1.6mm_P7.62mm_Horizontal" V 4030 5050 50  0001 C CNN
 F 3 "~" H 4100 5050 50  0001 C CNN
 	1    4100 5050
@@
 F 0 "R2" V 4200 5050 50  0000 C CNN
 F 1 "1k" V 4200 5200 50  0000 C CNN
-F 2 "" V 4030 5150 50  0001 C CNN
+F 2 "Resistor_THT:R_Axial_DIN0204_L3.6mm_D1.6mm_P7.62mm_Horizontal" V 4030 5150 50  0001 C CNN
 F 3 "~" H 4100 5150 50  0001 C CNN
 	1    4100 5150
@@
 F 0 "J3" H 7530 5192 50  0000 L CNN
 F 1 "Conn_01x03" H 7530 5101 50  0000 L CNN
-F 2 "" H 7450 5150 50  0001 C CNN
+F 2 "Connector_PinHeader_2.54mm:PinHeader_1x03_P2.54mm_Vertical" H 7450 5150 50  0001 C CNN
 F 3 "~" H 7450 5150 50  0001 C CNN
 	1    7450 5150
@@
 F 0 "R4" V 6450 5150 50  0000 C CNN
 F 1 "5k1" V 6450 5300 50  0000 C CNN
-F 2 "" V 6480 5250 50  0001 C CNN
+F 2 "Resistor_THT:R_Axial_DIN0204_L3.6mm_D1.6mm_P7.62mm_Horizontal" V 6480 5250 50  0001 C CNN
 F 3 "~" H 6550 5250 50  0001 C CNN
 	1    6550 5250
@@
 F 0 "C1" H 6750 5250 50  0000 L CNN
 F 1 "10u" H 6750 5150 50  0000 L CNN
-F 2 "" H 6988 5200 50  0001 C CNN
+F 2 "Resistor_THT:R_Axial_DIN0204_L3.6mm_D1.6mm_P5.08mm_Horizontal" H 6988 5200 50  0001 C CNN
 F 3 "~" H 6950 5350 50  0001 C CNN
 	1    6950 5350
@@
 F 0 "U2" H 10128 5396 50  0000 L CNN
 F 1 "GPS" H 10128 5305 50  0000 L CNN
-F 2 "" H 9800 5350 50  0001 C CNN
+F 2 "hitteStress21-pcb:GPS" H 9800 5350 50  0001 C CNN
 F 3 "" H 9800 5350 50  0001 C CNN
 	1    9800 5350
@@
 F 0 "R3" V 4200 5250 50  0000 C CNN
 F 1 "4R7" V 4200 5400 50  0000 C CNN
-F 2 "" V 4030 5350 50  0001 C CNN
+F 2 "Resistor_THT:R_Axial_DIN0204_L3.6mm_D1.6mm_P7.62mm_Horizontal" V 4030 5350 50  0001 C CNN
 F 3 "~" H 4100 5350 50  0001 C CNN
 	1    4100 5350

Commit message: Updates on footprints
Parts:
- added B1: LiPo_3V7, hitteStress21-pcb:LiPo_3V7_2000mAh_JST-PH, symbol HittStress21:LiPo_3V7
- J3: footprint Connector_PinHeader_2.54mm:PinHeader_1x03_P2.54mm_Vertical -> hitteStress21-pcb:Wurth_2109_p2.54
- PSU1: footprint Connector_PinHeader_2.54mm:PinHeader_1x03_P2.54mm_Vertical -> hitteStress21-pcb:MINIDCBOOST5V
Changed lines of the file:
@@
 F 0 "PSU1" H 1950 5665 50  0000 C CNN
 F 1 "MINIDCDCBOOST5V" H 1950 5574 50  0000 C CNN
-F 2 "Connector_PinHeader_2.54mm:PinHeader_1x03_P2.54mm_Vertical" H 1950 5250 50  0001 C CNN
+F 2 "hitteStress21-pcb:MINIDCBOOST5V" H 1950 5250 50  0001 C CNN
 F 3 "" H 1950 5250 50  0001 C CNN
 	1    1950 5250
@@
 5V_EXT
 Text Label 3450 5050 0    50   ~ 0
+SDS011_TX
+Text Label 3450 5150 0    50   ~ 0
 SDS011_RX
-Text Label 3450 5150 0    50   ~ 0
-SDS011_TX
 Text Notes 3700 4750 0    50   ~ 0
 Particlesensor SDS011
@@
 F 0 "J3" H 7530 5192 50  0000 L CNN
 F 1 "Conn_01x03" H 7530 5101 50  0000 L CNN
-F 2 "Connector_PinHeader_2.54mm:PinHeader_1x03_P2.54mm_Vertical" H 7450 5150 50  0001 C CNN
+F 2 "hitteStress21-pcb:Wurth_2109_p2.54" H 7450 5150 50  0001 C CNN
 F 3 "~" H 7450 5150 50  0001 C CNN
 	1    7450 5150
@@
 Wire Wire Line
 	3950 5350 3400 5350
+$Comp
+L HittStress21:LiPo_3V7 B1
+U 1 1 6003A431
+P 9600 2450
+F 0 "B1" H 9978 2496 50  0000 L CNN
+F 1 "LiPo_3V7" H 9978 2405 50  0000 L CNN
+F 2 "hitteStress21-pcb:LiPo_3V7_2000mAh_JST-PH" H 9600 2450 50  0001 C CNN
+F 3 "" H 9600 2450 50  0001 C CNN
+	1    9600 2450
+	1    0    0    -1
+$EndComp
 $EndSCHEMATC

Commit message: PCB design updates
Parts:
- added J4: Conn_01x02, hitteStress21-pcb:Wurth_2109_P2.54_2x1, symbol Connector_Generic:Conn_01x02
Connections:
- net labels removed: SDS011_RX, SDS011_TX
- wire segments 56 -> 59
Other:
- note added: "PV panel"
Changed lines of the file:
@@
 5V_EXT
 Text Label 3450 5050 0    50   ~ 0
-SDS011_TX
+SDS011_TXD
 Text Label 3450 5150 0    50   ~ 0
-SDS011_RX
+SDS011_RXD
 Text Notes 3700 4750 0    50   ~ 0
 Particlesensor SDS011
@@
 	1    0    0    -1
 $EndComp
+$Comp
+L Connector_Generic:Conn_01x02 J4
+U 1 1 600437D4
+P 4750 6450
+F 0 "J4" H 4830 6442 50  0000 L CNN
+F 1 "Conn_01x02" H 4830 6351 50  0000 L CNN
+F 2 "hitteStress21-pcb:Wurth_2109_P2.54_2x1" H 4750 6450 50  0001 C CNN
+F 3 "~" H 4750 6450 50  0001 C CNN
+	1    4750 6450
+	1    0    0    -1
+$EndComp
+Wire Wire Line
+	4550 6450 3400 6450
+Wire Wire Line
+	4550 6550 4400 6550
+Wire Wire Line
+	4400 6550 4400 6700
+$Comp
+L SparkFun-PowerSymbols:GND #GND0101
+U 1 1 60046B99
+P 4400 6700
+F 0 "#GND0101" H 4450 6650 45  0001 L BNN
+F 1 "GND" H 4400 6530 45  0000 C CNN
+F 2 "" H 4400 6600 60  0001 C CNN
+F 3 "" H 4400 6600 60  0001 C CNN
+	1    4400 6700
+	1    0    0    -1
+$EndComp
+Text Label 3450 6450 0    50   ~ 0
+PV
+Text Notes 4000 6250 0    50   ~ 0
+PV panel
 $EndSCHEMATC

Commit message: Added schema
Parts:
- B1: symbol HittStress21:LiPo_3V7 -> hitteStress21-pcb-rescue:LiPo_3V7-HittStress21
- PSU1: symbol HittStress21:MINIDCDCBOOST5V -> hitteStress21-pcb-rescue:MINIDCDCBOOST5V-HittStress21
- PSU2: symbol HittStress21:IRM-03 -> hitteStress21-pcb-rescue:IRM-03-HittStress21
- U1: symbol HittStress21:HTCC-AB01 -> hitteStress21-pcb-rescue:HTCC-AB01-HittStress21
- U2: symbol HittStress21:GPS -> hitteStress21-pcb-rescue:GPS-HittStress21
Changed lines of the file:
@@
 $EndDescr
 $Comp
-L HittStress21:IRM-03 PSU2
+L hitteStress21-pcb-rescue:IRM-03-HittStress21 PSU2
 U 1 1 5FFF7A4A
 P 3100 2000
@@
 $EndComp
 $Comp
-L HittStress21:MINIDCDCBOOST5V PSU1
+L hitteStress21-pcb-rescue:MINIDCDCBOOST5V-HittStress21 PSU1
 U 1 1 5FFF80A3
 P 1950 5250
@@
 $EndComp
 $Comp
-L SparkFun-PowerSymbols:GND #GND04
+L hitteStress21-pcb-rescue:GND-SparkFun-PowerSymbols #GND04
 U 1 1 5FFFEB8C
 P 5350 3100
@@
 $EndComp
 $Comp
-L SparkFun-PowerSymbols:GND #GND06
+L hitteStress21-pcb-rescue:GND-SparkFun-PowerSymbols #GND06
 U 1 1 5FFFF63E
 P 7550 3100
@@
 3V3
 $Comp
-L SparkFun-PowerSymbols:GND #GND01
+L hitteStress21-pcb-rescue:GND-SparkFun-PowerSymbols #GND01
 U 1 1 60000A77
 P 1950 5800
@@
 5V
 $Comp
-L SparkFun-PowerSymbols:GND #GND02
+L hitteStress21-pcb-rescue:GND-SparkFun-PowerSymbols #GND02
 U 1 1 60003428
 P 3600 2200
@@
 3V3_EXT
 $Comp
-L HittStress21:HTCC-AB01 U1
+L hitteStress21-pcb-rescue:HTCC-AB01-HittStress21 U1
 U 1 1 60009C11
 P 6450 2400
@@
 	4400 5250 4400 5550
 $Comp
-L SparkFun-PowerSymbols:GND #GND03
+L hitteStress21-pcb-rescue:GND-SparkFun-PowerSymbols #GND03
 U 1 1 60011F1B
 P 4400 5550
@@
 $EndComp
 $Comp
-L SparkFun-PowerSymbols:GND #GND05
+L hitteStress21-pcb-rescue:GND-SparkFun-PowerSymbols #GND05
 U 1 1 60021D16
 P 7150 5600
@@
 	7150 5550 7150 5600
 $Comp
-L HittStress21:GPS U2
+L hitteStress21-pcb-rescue:GPS-HittStress21 U2
 U 1 1 6003B0A4
 P 9800 5350
@@
 	9100 5250 9100 5800
 $Comp
-L SparkFun-PowerSymbols:GND #GND07
+L hitteStress21-pcb-rescue:GND-SparkFun-PowerSymbols #GND07
 U 1 1 6004350F
 P 9100 5800
@@
 	3950 5350 3400 5350
 $Comp
-L HittStress21:LiPo_3V7 B1
+L hitteStress21-pcb-rescue:LiPo_3V7-HittStress21 B1
 U 1 1 6003A431
 P 9600 2450
@@
 	4400 6550 4400 6700
 $Comp
-L SparkFun-PowerSymbols:GND #GND0101
+L hitteStress21-pcb-rescue:GND-SparkFun-PowerSymbols #GND0101
 U 1 1 60046B99
 P 4400 6700
